Commit message: robot size changed

File: double_robotics.urdf (robot description, URDF)
Before this commit: robot double_robotics, 7 links, 6 joints
Links:
- link base_link: geometry visual cylinder length=0.154 radius=0.0915
- link camera: geometry visual box size=0.08 0.01 0.022
- link ipad: geometry visual box size=0.204 0.01 0.2476
- link left_wheel: geometry visual cylinder length=0.051 radius=0.1115
- link right_wheel: geometry visual cylinder length=0.051 radius=0.1115
- link stick: geometry visual cylinder length=0.86 radius=0.025
Joints:
- joint base_to_left_wheel: origin xyz=-0.13 0 0 -> xyz=-0.1 0 0
- joint base_to_right_wheel: origin xyz=0.13 0 0 -> xyz=0.1 0 0
- joint base_to_stick: origin xyz=0 0 0.45 -> xyz=0 0 0.52
- joint ipad_to_camera: origin xyz=0 0 0.14 -> xyz=0 0 0.133
- joint stick_to_audio: origin xyz=0 0.04 0.19 -> xyz=0 0.04 0.29
- joint stick_to_ipad: origin xyz=0 0.03 0.35 -> xyz=0 0.03 0.45
